File: TSOC_PSoC4L/TSOC_PSoC4L.brd (EAGLE design)
At the start: 44.5 x 30.5 mm, 62 parts, among them U1 AP2112K-3.3V, U100 FM24W256-G, U2 MCP73831, U3 CY8C4247AZI-L433, Y100 3.2768KHZ

Commit message: update to Rev1.2
Parts:
- removed $$U$1, $$U$2: TSOC-LOGO-SMALL, thingSoC:TSOC-LOGO-SML
- added C103: 100nf, Seeed-Capacitor-2016:C0603
- added C17: 47uf, Seeed-Capacitor-2016:AVX-A
- R7: value 1K 1/10W -> 0R
- moved U$100 1.14 mm to (30.0, 11.7)
- renumbered OSC to Y101
Connections:
- net 5V0: now also JTAG.12
- net GND: now also C103.2, C17.-
- net VCC: now also C103.1, C17.+; no longer JTAG.12
Routing:
- net 5V0: track 67.6 -> 79.2 mm
- net GND: track 263.7 -> 271.5 mm, vias 11 -> 13
- net VCC: track 52.6 -> 59.2 mm
- net !XRES: vias 2 -> 4
Other:
- board text added: "(Optional NVSRAM, Crystal, Oscillator)"
- board text added: "CY8C4247AZI-L433"
- board text added: "Model: TSOC_PSOC4L"
- board text added: "PatternAgents thingSoC!"
- board text added: "Rev. 1.2"
- board text removed: "(Optional I2C NVSRAM)"
- board text removed: "(Optional Oscillators)"
- board text removed: "Rev. 1.0"

Commit message: update to Rev1.2
Parts:
- removed R7: 0R, Seeed-Resistor-2016:R0603
Connections:
- removed net P13_2: R7.1, U3.25
- net VBUS: now also U3.25; no longer R7.2
Routing:
- net P13_2: track 25.8 -> 0.00 mm, vias 2 -> 0
- net VBUS: track 43.3 -> 68.7 mm, vias 2 -> 4
- net VCC: track 59.2 -> 64.7 mm
- net GND: track 271.5 -> 275.6 mm
- net 5V0: track 79.2 -> 76.5 mm
Other:
- board text added: "VCC/5V0"
- board text removed: "VCC/VCC"
