File: TSOC_PSoC4L/TSOC_PSoC4L.sch (EAGLE design)
At the start: 61 parts, among them U1 AP2112K-3.3V, U100 FM24W256-G, U2 MCP73831, U3 CY8C4247AZI-L433, Y100 3.2768KHZ

Commit message: update to Rev1.2
Parts:
- removed $$U$1, $$U$2: TSOC-LOGO-SMALL, thingSoC:TSOC-LOGO-SMALL
- added C103: 100nf, Seeed-Capacitor-2016:CERAMIC-100NF-50V-10%-X7R(0603)
- added C17: 47uf, Seeed-Capacitor-2016:TANTALUM-SMD-47UF-6.3V(AVX-A)
- R7: value 1K 1/10W -> 0R; device Seeed-Resistor-2016:SMD-RES-1K-5%-1/10W(0603) -> Seeed-Resistor-2016:SMD-RES-0R-5%-1/10W(0603)
- renumbered OSC to Y101
Connections:
- net 5V0: now also JTAG.12
- net GND: now also C103.2, C17.-
- net VCC: now also C103.1, C17.+; no longer JTAG.12
Changed lines of the file:
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@@
 <part name="RESET" library="Seeed-Switch-2016" deviceset="SMD-BUTTON(2P-3.0X2.5X1.2+0.4MM)" device="-B3U-1000P-2P-SMD" value="B3U-1000P-2P-SMD"/>
 <part name="USER" library="Seeed-Switch-2016" deviceset="SMD-BUTTON(2P-3.0X2.5X1.2+0.4MM)" device="-B3U-1000P-2P-SMD" value="B3U-1000P-2P-SMD"/>
-<part name="R7" library="Seeed-Resistor-2016" deviceset="SMD-RES-1K-5%-1/10W(0603)" device="" value="1K 1/10W"/>
+<part name="R7" library="Seeed-Resistor-2016" deviceset="SMD-RES-0R-5%-1/10W(0603)" device="" value="0R"/>
 <part name="U$5" library="PatternAgents-Beautify" deviceset="GND" device=""/>
-<part name="$$U$2" library="thingSoC" deviceset="TSOC-LOGO" device="-SMALL"/>
 <part name="Y100" library="Seeed-Crystal Oscillator-2016" deviceset="SMD-CRYSTAL-32.768KHZ-12.5PF-20PPM-90K(2P-L2.0X1.2MM)" device="" value="3.2768KHZ"/>
 <part name="C101" library="Seeed-Capacitor-2016" deviceset="CERAMIC-12PF-50V-5%-NPO(0603)" device="" value="12pf"/>
@@
 <part name="GND21" library="supply1" deviceset="GND" device=""/>
 <part name="GND22" library="supply1" deviceset="GND" device=""/>
-<part name="OSC" library="SparkFun-FreqCtrl" deviceset="OSCILLATOR" device="5X3"/>
+<part name="Y101" library="SparkFun-FreqCtrl" deviceset="OSCILLATOR" device="5X3"/>
 <part name="GND24" library="supply1" deviceset="GND" device=""/>
 <part name="U100" library="PatternAgents-Cypress" deviceset="FM24W256" device="-G"/>
@@
 <part name="U$21" library="PatternAgents-Beautify" deviceset="GND" device=""/>
 <part name="U$24" library="PatternAgents-Beautify" deviceset="GND" device=""/>
-<part name="$$U$1" library="thingSoC" deviceset="TSOC-LOGO" device="-SMALL"/>
+<part name="C103" library="Seeed-Capacitor-2016" deviceset="CERAMIC-100NF-50V-10%-X7R(0603)" device="" value="100nf"/>
+<part name="GND4" library="supply1" deviceset="GND" device=""/>
+<part name="C17" library="Seeed-Capacitor-2016" deviceset="TANTALUM-SMD-47UF-6.3V(AVX-A)" device="" value="47uf"/>
+<part name="U$6" library="PatternAgents-Beautify" deviceset="GND" device=""/>
 </parts>
 <sheets>
@@
 <instance part="R7" gate="G$1" x="401.32" y="88.9" rot="R180"/>
 <instance part="U$5" gate="G$1" x="140.97" y="276.86"/>
-<instance part="$$U$2" gate="G$1" x="461.01" y="247.65"/>
 <instance part="Y100" gate="G$1" x="58.42" y="261.62" rot="MR0"/>
 <instance part="C101" gate="G$1" x="71.12" y="251.46" rot="MR270"/>
@@
 <instance part="GND21" gate="1" x="71.12" y="241.3"/>
 <instance part="GND22" gate="1" x="48.26" y="241.3"/>
-<instance part="OSC" gate="G$1" x="114.3" y="254"/>
+<instance part="Y101" gate="G$1" x="114.3" y="254"/>
 <instance part="GND24" gate="1" x="129.54" y="243.84" rot="MR0"/>
 <instance part="U100" gate="G$1" x="415.29" y="327.66" smashed="yes">
@@
 <instance part="U$21" gate="G$1" x="440.69" y="317.5"/>
 <instance part="U$24" gate="G$1" x="393.7" y="314.96"/>
-<instance part="$$U$1" gate="G$1" x="459.74" y="29.21"/>
+<instance part="C103" gate="G$1" x="93.98" y="251.46" rot="MR270"/>
+<instance part="GND4" gate="1" x="93.98" y="241.3" rot="MR0"/>
+<instance part="C17" gate="G$1" x="433.07" y="156.21" rot="R270"/>
+<instance part="U$6" gate="G$1" x="433.07" y="147.32"/>
 </instances>
 <busses>
@@
 </segment>
 <segment>
-<pinref part="OSC" gate="G$1" pin="GND"/>
+<pinref part="Y101" gate="G$1" pin="GND"/>
 <pinref part="GND24" gate="1" pin="GND"/>
 <wire x1="127" y1="251.46" x2="129.54" y2="251.46" width="0.1524" layer="91"/>
@@
 <junction x="402.59" y="325.12"/>
 </segment>
+<segment>
+<pinref part="GND4" gate="1" pin="GND"/>
+<pinref part="C103" gate="G$1" pin="2"/>
+<wire x1="93.98" y1="243.84" x2="93.98" y2="247.65" width="0.1524" layer="91"/>
+</segment>
+<segment>
+<pinref part="C17" gate="G$1" pin="-"/>
+<pinref part="U$6" gate="G$1" pin="GND"/>
+<wire x1="433.07" y1="152.4" x2="433.07" y2="147.32" width="0.1524" layer="91"/>
+</segment>
 </net>
 <net name="P1_2" class="0">
@@
 </segment>
 <segment>
-<pinref part="OSC" gate="G$1" pin="OUT"/>
+<pinref part="Y101" gate="G$1" pin="OUT"/>
 <wire x1="127" y1="256.54" x2="132.08" y2="256.54" width="0.1524" layer="91"/>
 <label x="132.08" y="256.54" size="1.4224" layer="95" font="vector" ratio="10" xref="yes"/>
@@
 <wire x1="406.4" y1="185.42" x2="406.4" y2="193.04" width="0.1524" layer="91"/>
 <junction x="406.4" y="193.04"/>
+</segment>
+<segment>
+<wire x1="144.78" y1="149.86" x2="154.94" y2="149.86" width="0.1524" layer="91"/>
+<label x="154.94" y="149.86" size="1.27" layer="95" font="vector" ratio="10" rot="MR180" xref="yes"/>
+<pinref part="JTAG" gate="G$1" pin="12"/>
 </segment>
 </net>
@@
 </segment>
 <segment>
-<wire x1="144.78" y1="149.86" x2="154.94" y2="149.86" width="0.1524" layer="91"/>
-<label x="154.94" y="149.86" size="1.27" layer="95" font="vector" ratio="10" rot="MR180" xref="yes"/>
-<pinref part="JTAG" gate="G$1" pin="12"/>
-</segment>
-<segment>
 <pinref part="L2" gate="L" pin="1"/>
-<wire x1="426.72" y1="182.88" x2="441.96" y2="182.88" width="0.1524" layer="91"/>
+<wire x1="426.72" y1="182.88" x2="433.07" y2="182.88" width="0.1524" layer="91"/>
+<wire x1="433.07" y1="182.88" x2="441.96" y2="182.88" width="0.1524" layer="91"/>
 <wire x1="452.12" y1="182.88" x2="441.96" y2="182.88" width="0.1524" layer="91"/>
 <pinref part="L1" gate="L" pin="1"/>
@@
 <junction x="441.96" y="193.04"/>
 <label x="436.88" y="193.04" size="1.27" layer="95" font="vector" ratio="10" rot="R180" xref="yes"/>
-</segment>
-<segment>
-<pinref part="OSC" gate="G$1" pin="VCC"/>
+<pinref part="C17" gate="G$1" pin="+"/>
+<wire x1="433.07" y1="160.02" x2="433.07" y2="182.88" width="0.1524" layer="91"/>
+<junction x="433.07" y="182.88"/>
+</segment>
+<segment>
+<pinref part="Y101" gate="G$1" pin="VCC"/>
 <wire x1="101.6" y1="256.54" x2="99.06" y2="256.54" width="0.1524" layer="91"/>
-<pinref part="OSC" gate="G$1" pin="EN"/>
-<wire x1="99.06" y1="256.54" x2="96.52" y2="256.54" width="0.1524" layer="91"/>
+<pinref part="Y101" gate="G$1" pin="EN"/>
+<wire x1="99.06" y1="256.54" x2="93.98" y2="256.54" width="0.1524" layer="91"/>
+<wire x1="93.98" y1="256.54" x2="88.9" y2="256.54" width="0.1524" layer="91"/>
 <wire x1="101.6" y1="251.46" x2="99.06" y2="251.46" width="0.1524" layer="91"/>
 <wire x1="99.06" y1="251.46" x2="99.06" y2="256.54" width="0.1524" layer="91"/>
 <junction x="99.06" y="256.54"/>
-<label x="96.52" y="256.54" size="1.4224" layer="95" font="vector" ratio="10" rot="R180" xref="yes"/>
-</segment>
-<segment>
+<label x="88.9" y="256.54" size="1.4224" layer="95" font="vector" ratio="10" rot="R180" xref="yes"/>
+<pinref part="C103" gate="G$1" pin="1"/>
+<wire x1="93.98" y1="255.27" x2="93.98" y2="256.54" width="0.1524" layer="91"/>
+<junction x="93.98" y="256.54"/>
+</segment>
+<segment>

Commit message: update to Rev1.2
Parts:
- removed R7: 0R, Seeed-Resistor-2016:SMD-RES-0R-5%-1/10W(0603)
Connections:
- removed net P13_2: R7.1, U3.VBUS
- net VBUS: now also U3.VBUS; no longer R7.2
Changed lines of the file:
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@@
 <part name="RESET" library="Seeed-Switch-2016" deviceset="SMD-BUTTON(2P-3.0X2.5X1.2+0.4MM)" device="-B3U-1000P-2P-SMD" value="B3U-1000P-2P-SMD"/>
 <part name="USER" library="Seeed-Switch-2016" deviceset="SMD-BUTTON(2P-3.0X2.5X1.2+0.4MM)" device="-B3U-1000P-2P-SMD" value="B3U-1000P-2P-SMD"/>
-<part name="R7" library="Seeed-Resistor-2016" deviceset="SMD-RES-0R-5%-1/10W(0603)" device="" value="0R"/>
 <part name="U$5" library="PatternAgents-Beautify" deviceset="GND" device=""/>
 <part name="Y100" library="Seeed-Crystal Oscillator-2016" deviceset="SMD-CRYSTAL-32.768KHZ-12.5PF-20PPM-90K(2P-L2.0X1.2MM)" device="" value="3.2768KHZ"/>
@@
 <attribute name="VALUE" x="147.32" y="295.91" size="1.27" layer="96" ratio="10"/>
 </instance>
-<instance part="R7" gate="G$1" x="401.32" y="88.9" rot="R180"/>
 <instance part="U$5" gate="G$1" x="140.97" y="276.86"/>
 <instance part="Y100" gate="G$1" x="58.42" y="261.62" rot="MR0"/>
@@
 <net name="VBUS" class="0">
 <segment>
-<pinref part="D1" gate="G$1" pin="+"/>
-<wire x1="388.62" y1="101.6" x2="394.97" y2="101.6" width="0.1524" layer="91"/>
-<wire x1="388.62" y1="101.6" x2="388.62" y2="88.9" width="0.1524" layer="91"/>
-<wire x1="388.62" y1="88.9" x2="397.51" y2="88.9" width="0.1524" layer="91"/>
-<pinref part="R7" gate="G$1" pin="2"/>
-<wire x1="388.62" y1="88.9" x2="388.62" y2="81.28" width="0.1524" layer="91"/>
-<junction x="388.62" y="88.9"/>
-<wire x1="388.62" y1="81.28" x2="411.48" y2="81.28" width="0.1524" layer="91"/>
-<label x="411.48" y="81.28" size="1.27" layer="95" font="vector" ratio="10" xref="yes"/>
-<pinref part="USB" gate="G$1" pin="VBUS"/>
-<wire x1="342.9" y1="101.6" x2="388.62" y2="101.6" width="0.1524" layer="91"/>
-<junction x="388.62" y="101.6"/>
-</segment>
-<segment>
 <label x="411.48" y="40.64" size="1.27" layer="95" font="vector" ratio="10" xref="yes"/>
 <wire x1="403.86" y1="31.75" x2="403.86" y2="40.64" width="0.1524" layer="91"/>
@@
 <pinref part="C6" gate="G$1" pin="1"/>
 <pinref part="LED2" gate="G$1" pin="+"/>
+</segment>
+<segment>
+<pinref part="U3" gate="U1" pin="VBUS"/>
+<wire x1="114.3" y1="327.66" x2="139.7" y2="327.66" width="0.1524" layer="91"/>
+<label x="139.7" y="327.66" size="1.27" layer="95" font="vector" ratio="10" xref="yes"/>
+</segment>
+<segment>
+<label x="411.48" y="88.9" size="1.27" layer="95" font="vector" ratio="10" xref="yes"/>
+<pinref part="D1" gate="G$1" pin="+"/>
+<wire x1="388.62" y1="101.6" x2="394.97" y2="101.6" width="0.1524" layer="91"/>
+<wire x1="388.62" y1="101.6" x2="388.62" y2="88.9" width="0.1524" layer="91"/>
+<pinref part="USB" gate="G$1" pin="VBUS"/>
+<wire x1="342.9" y1="101.6" x2="388.62" y2="101.6" width="0.1524" layer="91"/>
+<junction x="388.62" y="101.6"/>
+<wire x1="411.48" y1="88.9" x2="388.62" y2="88.9" width="0.1524" layer="91"/>
 </segment>
 </net>
@@
 </segment>
 </net>
-<net name="P13_2" class="0">
-<segment>
-<pinref part="U3" gate="U1" pin="VBUS"/>
-<wire x1="114.3" y1="327.66" x2="139.7" y2="327.66" width="0.1524" layer="91"/>
-<label x="139.7" y="327.66" size="1.27" layer="95" font="vector" ratio="10" xref="yes"/>
-</segment>
-<segment>
-<pinref part="R7" gate="G$1" pin="1"/>
-<wire x1="405.13" y1="88.9" x2="411.48" y2="88.9" width="0.1524" layer="91"/>
-<label x="411.48" y="88.9" size="1.27" layer="95" font="vector" ratio="10" xref="yes"/>
-</segment>
-</net>
