File: TSOC_PSoC4L/revisions/R1_2/TSOC_PSoC4L.brd (EAGLE design)
At the start: 44.5 x 30.5 mm, 62 parts, among them U1 AP2112K-3.3V, U100 FM24W256-G, U2 MCP73831, U3 CY8C4247AZI-L433, Y100 3.2768KHZ, Y101 OSCILLATOR5X3

Commit message: update to Rev1.2
Parts:
- removed R7: 0R, Seeed-Resistor-2016:R0603
Connections:
- removed net P13_2: R7.1, U3.25
- net VBUS: now also U3.25; no longer R7.2
Routing:
- net P13_2: track 25.8 -> 0.00 mm, vias 2 -> 0
- net VBUS: track 43.3 -> 68.7 mm, vias 2 -> 4
- net VCC: track 59.2 -> 64.7 mm
- net GND: track 271.5 -> 275.6 mm
- net 5V0: track 79.2 -> 76.5 mm
Other:
- board text added: "VCC/5V0"
- board text removed: "VCC/VCC"
